File: Schaltplan.kicad_sch (KiCad schematic)
At the start: 17 parts, among them K1 Relay, P1 USB Port vorheriger, P2 USB Port nächster, P4 USB Port Laden, U1 DC DC Wandler, U2 DC DC Wandler, U3 DS18B20, U4 Display, U5 DC DC Wandler, U6 Digitaler Poti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

Commit message: Cable move
Co-authored-by: JumpStone <hi@jumpstone4477.de>
Connections:
- net at K1. (NC): now also A1.7 (D4)
Changed lines of the file:
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@@
+	)
+	(junction
+		(at 20.32 58.42)
+		(diameter 0)
+		(color 0 0 0 0)
 	)
 	(junction
@@
 	)
 	(junction
-		(at 17.78 58.42)
-		(diameter 0)
-		(color 0 0 0 0)
-	)
-	(junction
 		(at 60.96 147.32)
 		(diameter 0)
@@
 	(wire
 		(pts
-			(xy 17.78 35.56) (xy 29.21 35.56)
+			(xy 20.32 35.56) (xy 29.21 35.56)
 		)
 		(stroke
@@
 	(wire
 		(pts
-			(xy 29.21 58.42) (xy 17.78 58.42)
+			(xy 29.21 58.42) (xy 20.32 58.42)
 		)
 		(stroke
@@
 	(wire
 		(pts
-			(xy 21.59 15.24) (xy 29.21 15.24)
+			(xy 22.86 15.24) (xy 29.21 15.24)
+		)
+		(stroke
+			(width 0)
+			(type default)
+		)
+	)
+	(wire
+		(pts
+			(xy 20.32 58.42) (xy 20.32 130.81)
 		)
 		(stroke
@@
 	(wire
 		(pts
-			(xy 17.78 35.56) (xy 17.78 58.42)
+			(xy 20.32 35.56) (xy 20.32 58.42)
 		)
 		(stroke
@@
 	(wire
 		(pts
-			(xy 21.59 36.83) (xy 21.59 15.24)
+			(xy 22.86 36.83) (xy 22.86 15.24)
 		)
 		(stroke
@@
 	(wire
 		(pts
-			(xy 17.78 130.81) (xy 20.32 130.81)
-		)
-		(stroke
-			(width 0)
-			(type default)
-		)
-	)
-	(wire
-		(pts
 			(xy 134.62 58.42) (xy 134.62 92.71)
 		)
@@
 	(wire
 		(pts
-			(xy 17.78 58.42) (xy 17.78 130.81)
-		)
-		(stroke
-			(width 0)
-			(type default)
-		)
-	)
-	(wire
-		(pts
 			(xy 118.11 186.69) (xy 118.11 191.77)
 		)
@@
 	(wire
 		(pts
-			(xy 29.21 36.83) (xy 21.59 36.83)
-		)
-		(stroke
+			(xy 29.21 36.83) (xy 22.86 36.83)
+		)
+		(stroke
